File: Atari65XEC070067RevB.kicad_pcb (KiCad board)
At the start: 2 copper layers, 322 x 204.1 mm, 341 parts, among them J2 MONITOR, J5 JOY1, J6 JOY1, J7 DIN-7, J8 KEYBOARD, Q1 2N3904, Q2 2N3904, Q3 2N3904, Q4 2N3904, Q5 2N3904, Q6 2N3904, Q7 MPSA55, SW1 SW_SPDT, U1 LM358, U10 4164, U11 4164, U12 4164, U13 4164, U14 4164, U15 4164, U16 4164, U17 C014889/GTIA, U18 74LS08, U19 NE555P, U2 74LS138, U20 4050, U21 74LS74, U22 C012294/POKEY, U23 C014795 PIA/6520, U24 4051, U25 4051, U26 4164, U27 4164, U28 4164, U29 4164, U3 MMU, U30 4164, U31 4164, U32 4164, U33 4164, U34 MMMU, U35 74LS95, U4 BASIC, U5 OS ROM, U6 CO14806/SALLY, U7 C021698/ANTIC, U8 C061991/FREDDIE, U9 4164, Y2 4.33618MHz

Commit message: fix din ports
Parts:
- J7: footprint Library:CUI_SDS-70J -> Library:CUI_SDS-70J_Atari
- moved R52 12.6 mm to (151.1, 76.7), turned to -90 degrees
- moved J7 1.92 mm to (87.9, 50.0)
- moved C16 0.25 mm to (107.8, 97.8)
- moved R53 0.10 mm to (154.4, 89.4)
Routing:
- net /MONITOR_AUDIO: track 0.00 -> 99.7 mm
- net GND: track 676.3 -> 772.1 mm
- net /CHROMA: track 0.00 -> 80.1 mm, vias 0 -> 1
- net Net-(A1-Pad1): track 93.5 -> 42.9 mm
- net A9: track 175.0 -> 223.3 mm, vias 1 -> 2
- net A11: track 205.1 -> 248.0 mm, vias 3 -> 4
- net /LUMA: track 0.00 -> 36.4 mm
- net A8: track 201.7 -> 236.6 mm, vias 2 -> 3
- net /COMPOSITE: track 0.00 -> 31.2 mm
- net D4: track 242.4 -> 271.2 mm
- net D5: track 271.7 -> 300.0 mm
- net D6: track 268.9 -> 297.2 mm
- net /BO2: track 88.7 -> 116.2 mm
- net D1: track 363.8 -> 390.7 mm
- net D3: track 230.6 -> 257.2 mm
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