File: Atari65XEC070067RevB.kicad_pcb (KiCad board)
At the start: 2 copper layers, 322 x 204.1 mm, 340 parts, among them J1 SIO, J2 MONITOR, J5 JOY1, J6 JOY1, J7 DIN-7, J8 KEYBOARD, Q1 2N3904, Q2 2N3904, Q3 2N3904, Q4 2N3904, Q5 2N3904, Q6 2N3904, Q7 MPSA55, SW1 SW_SPDT, U1 LM358, U10 4164, U11 4164, U12 4164, U13 4164, U14 4164, U15 4164, U16 4164, U17 C014889/GTIA, U18 74LS08, U19 NE555P, U2 74LS138, U20 4050, U21 74LS74, U22 C012294/POKEY, U23 C014795 PIA/6520, U24 4051, U25 4051, U26 4164, U27 4164, U28 4164, U29 4164, U3 MMU, U30 4164, U31 4164, U32 4164, U33 4164, U34 MMMU, U35 74LS95, U4 BASIC, U5 OS ROM, U6 C061991/FREDDIE, U7 C021698/ANTIC, U8 CO14806/SALLY, U9 4164, Y2 4.33618MHz

Commit message: progress routing
Parts:
- moved R42 5.08 mm to (171.4, 157.4)
- moved R44 5.08 mm to (176.5, 157.4)
- moved C44 0.48 mm to (181.7, 109.7)
- moved R35 0.48 mm to (181.7, 112.5)
- moved R201 0.30 mm to (154.8, 160.5)
Connections:
- net /PB7 renamed Net-(U23-PB7)
- U20 pad 16: (no net) -> +5VA
- U20 pad 9: unconnected-(U20-Pad9) -> GND
Routing:
- net +5VA: track 1829.7 -> 1987.0 mm
- net /SIO_AUDIO: track 51.2 -> 167.5 mm, vias 0 -> 4
- net A2: track 310.9 -> 415.5 mm, vias 5 -> 6
- net A1: track 357.6 -> 453.1 mm, vias 5 -> 6
- net Net-(U23-PB7): track 11.9 -> 74.8 mm
- net A4: track 281.9 -> 342.4 mm, vias 3 -> 4
- net A3: track 300.3 -> 359.6 mm
- net /RD5: track 149.3 -> 206.0 mm, vias 4 -> 5
- net A5: track 237.4 -> 292.6 mm, vias 2 -> 3
- net Net-(U17-CADJ): track 95.1 -> 150.2 mm, vias 3 -> 4
- net Net-(C19-Pad2): track 66.2 -> 120.6 mm, vias 1 -> 2
- net A8: track 263.1 -> 310.3 mm
- net D4: track 425.4 -> 472.5 mm
- net Net-(U8-O0): track 40.8 -> 87.6 mm, vias 1 -> 2
- net A6: track 242.3 -> 279.7 mm
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