File: Atari65XEC070067RevB.kicad_pcb (KiCad board)
At the start: 2 copper layers, 323.9 x 204 mm, 362 parts, among them J1 SIO, J2 MONITOR, J5 JOY1, J6 JOY1, J7 DIN-7, J8 KEYBOARD, Q1 2N3904, Q2 2N3904, Q3 2N3904, Q4 2N3904, Q5 2N3904, Q6 2N3904, Q7 MPSA55, SW1 SW_SPDT, U1 LM358, U10 4164, U11 4164, U12 4164, U13 4164, U14 4164, U15 4164, U16 4164, U17 C014889/GTIA, U18 74LS08, U19 NE555P, U2 74LS138, U20 4050, U21 74LS74, U22 C012294/POKEY, U23 C014795 PIA/6520, U24 4051, U25 4051, U26 4164, U27 4164, U28 4164, U29 4164, U3 MMU, U30 4164, U31 4164, U32 4164, U33 4164, U34 MMMU, U35 74LS95, U4 BASIC, U5 OS ROM, U6 C061991/FREDDIE, U7 C021698/ANTIC, U8 CO14806/SALLY, U9 4164, Y2 4.33618MHz

Commit message: tidy up schematic
Parts:
- removed QR*****: https://github.com/jimbro1000/Atari65_130XE_C070067, Library:barcode
- CR2, CR4, CR5: value ~ -> 1N4148
- R128, R129, R130, R131, R90: value 100 -> 100R
Connections:
- JA4 pad S: /BO2 -> /Bphi2
- R20 pad 1: /Bphi2 -> /phi2
- U17 pad 30: /BO2 -> /Bphi2
- U18 pad 1: /Bphi2 -> /phi2
- U18 pad 3: /BO2 -> /Bphi2
- U22 pad 7: /BO2 -> /Bphi2
- U23 pad 25: /BO2 -> /Bphi2
- U34 pad 19: /Bphi2 -> /phi2
- U35 pad 9: /BO2 -> /Bphi2
- U6 pad 5: /Bphi2 -> /phi2
- U7 pad 29: /BO2 -> /Bphi2
- U8 pad 39: /Bphi2 -> /phi2
Routing:
- net /phi2: track 0.00 -> 449.5 mm, vias 0 -> 6
- net /BO2: track 421.0 -> 0.00 mm, vias 4 -> 0
- net /Bphi2: track 449.5 -> 421.0 mm, vias 6 -> 4
