File: Atari65XEC070067RevB.kicad_sch (KiCad schematic)
At the start: 341 parts, among them J1 SIO, J2 MONITOR, J5 JOY1, J6 JOY1, J7 DIN-7, J8 KEYBOARD, Q1 2N3904, Q2 2N3904, Q3 2N3904, Q4 2N3904, Q5 2N3904, Q6 2N3904, Q7 MPSA55, SW1 SW_SPDT, U1 LM358, U10 4164, U11 4164, U12 4164, U13 4164, U14 4164, U15 4164, U16 4164, U17 C014889/GTIA, U18 74LS08, U19 NE555P, U2 74LS138, U20 4050, U21 74LS74, U22 C012294/POKEY, U23 C014795 PIA/6520, U24 4051, U25 4051, U26 4164, U27 4164, U28 4164, U29 4164, U3 MMU, U30 4164, U31 4164, U32 4164, U33 4164, U34 MMMU, U35 74LS95, U4 BASIC, U5 OS ROM, U6 C061991/FREDDIE, U7 C021698/ANTIC, U8 CO14806/SALLY, U9 4164, Y2 4.33618MHz

Commit message: progress routing
Parts:
- added R88: 3k, Library:R_Axial_L9.0mm_D2.7mm_P12.70mm_Horizontal, symbol Device:R_Small
Connections:
- net Case is gone; now on net GND: A1.6 (Case)
- net +5VA: now also C43.1, U18.14 (VCC), R88.2
- net +5VC: no longer C43.1, U18.14 (VCC)
- net PB0: now also R88.1
- net at R200.2, U19.2 (TR): now also C200.1, U19.6 (THR)
- net at U19.7 (DIS): no longer C200.1
Other:
- moved on the sheet: C200, R40
Changed lines of the file:
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@@
 	)
 	(junction
+		(at 284.48 201.93)
+		(diameter 0)
+		(color 0 0 0 0)
+	)
+	(junction
 		(at 280.67 279.4)
 		(diameter 0)
@@
 	)
 	(junction
-		(at 292.1 199.39)
-		(diameter 0)
-		(color 0 0 0 0)
-	)
-	(junction
 		(at 34.29 76.2)
 		(diameter 0)
@@
 	)
 	(junction
+		(at 292.1 201.93)
+		(diameter 0)
+		(color 0 0 0 0)
+	)
+	(junction
 		(at 422.91 341.63)
 		(diameter 0)
@@
 	)
 	(junction
+		(at 266.7 201.93)
+		(diameter 0)
+		(color 0 0 0 0)
+	)
+	(junction
 		(at 234.95 271.78)
 		(diameter 0)
@@
 	)
 	(junction
+		(at 414.02 162.56)
+		(diameter 0)
+		(color 0 0 0 0)
+	)
+	(junction
 		(at 232.41 156.21)
 		(diameter 0)
@@
 	)
 	(no_connect
-		(at 284.48 201.93)
-	)
-	(no_connect
 		(at 345.44 67.31)
 	)
@@
 		(at 276.86 120.65)
 	)
+	(no_connect
+		(at 284.48 199.39)
+	)
 	(bus_entry
 		(at 128.27 266.7)
@@
 	(wire
 		(pts
+			(xy 284.48 201.93) (xy 284.48 210.82)
+		)
+		(stroke
+			(width 0)
+			(type default)
+		)
+	)
+	(wire
+		(pts
 			(xy 72.39 284.48) (xy 55.88 284.48)
 		)
@@
 	(wire
 		(pts
-			(xy 290.83 199.39) (xy 292.1 199.39)
+			(xy 290.83 201.93) (xy 292.1 201.93)
 		)
 		(stroke
@@
 	(wire
 		(pts
-			(xy 284.48 199.39) (xy 285.75 199.39)
-		)
-		(stroke
-			(width 0)
-			(type default)
-		)
-	)
-	(wire
-		(pts
 			(xy 30.48 314.96) (xy 64.77 314.96)
 		)
@@
 	(wire
 		(pts
-			(xy 292.1 195.58) (xy 292.1 199.39)
+			(xy 284.48 210.82) (xy 266.7 210.82)
 		)
 		(stroke
@@
 	(wire
 		(pts
-			(xy 414.02 48.26) (xy 414.02 173.99)
+			(xy 414.02 48.26) (xy 414.02 162.56)
 		)
 		(stroke
@@
 	(wire
 		(pts
+			(xy 414.02 162.56) (xy 416.56 162.56)
+		)
+		(stroke
+			(width 0)
+			(type default)
+		)
+	)
+	(wire
+		(pts
 			(xy 535.94 275.59) (xy 535.94 341.63)
 		)
@@
 	(wire
 		(pts
+			(xy 266.7 210.82) (xy 266.7 201.93)
+		)
+		(stroke
+			(width 0)
+			(type default)
+		)
+	)
+	(wire
+		(pts
 			(xy 420.37 328.93) (xy 422.91 328.93)
 		)
@@
 	(wire
 		(pts
-			(xy 292.1 199.39) (xy 292.1 203.2)
-		)
-		(stroke
-			(width 0)
-			(type default)
-		)
-	)
-	(wire
-		(pts
 			(xy 226.06 289.56) (xy 234.95 289.56)
 		)
@@
 	(wire
 		(pts
+			(xy 292.1 195.58) (xy 292.1 201.93)
+		)
+		(stroke
+			(width 0)
+			(type default)
+		)
+	)
+	(wire
+		(pts
 			(xy 226.06 82.55) (xy 226.06 77.47)
 		)
@@
 	(wire
 		(pts
+			(xy 284.48 201.93) (xy 285.75 201.93)
+		)
+		(stroke
+			(width 0)
+			(type default)
+		)
+	)
+	(wire
+		(pts
 			(xy 218.44 271.78) (xy 226.06 271.78)
 		)
@@
 	(wire
 		(pts
-			(xy 292.1 208.28) (xy 292.1 236.22)
+			(xy 292.1 214.63) (xy 292.1 236.22)
 		)
 		(stroke
@@
 	(wire
 		(pts
+			(xy 414.02 162.56) (xy 414.02 173.99)
+		)
+		(stroke
+			(width 0)
+			(type default)
+		)
+	)
+	(wire
+		(pts
 			(xy 187.96 99.06) (xy 187.96 43.18)
 		)
@@
 	(wire
 		(pts
+			(xy 292.1 201.93) (xy 292.1 209.55)
+		)
+		(stroke
+			(width 0)
+			(type default)
+		)
+	)
+	(wire
+		(pts
 			(xy 60.96 149.86) (xy 60.96 292.1)
 		)
@@
 	(symbol
 		(lib_id "Device:R_Small")
-		(at 292.1 205.74 0)
+		(at 292.1 212.09 0)
 		(unit 1)
 		(exclude_from_sim no)
@@
 		(dnp no)
 		(property "Reference" "R40"
-			(at 293.624 205.74 0)
+			(at 293.624 212.09 0)
 			(effects
 				(font
@@
 		)
 		(property "Value" "100R"
-			(at 293.624 208.28 0)
+			(at 293.624 214.63 0)
 			(effects
 				(font
@@
 		)
 		(property "Footprint" "Library:R_Axial_L9.0mm_D2.7mm_P12.70mm_Horizontal"
-			(at 292.1 205.74 0)
+			(at 292.1 212.09 0)
 			(effects
 				(font
@@
 		)
 		(property "Datasheet" "~"
-			(at 292.1 205.74 0)
+			(at 292.1 212.09 0)
 			(effects
 				(font
@@
 		)
 		(property "Description" "Resistor, small symbol"
-			(at 292.1 205.74 0)
+			(at 292.1 212.09 0)
 			(effects
 				(font
@@
 	)
 	(symbol
+		(lib_id "power:+5VA")
+		(at 421.64 162.56 270)
+		(unit 1)
+		(exclude_from_sim no)
+		(in_bom yes)
+		(on_board yes)
+		(dnp no)
+		(fields_autoplaced yes)
+		(property "Reference" "#PWR0186"
+			(at 417.83 162.56 0)
+			(effects
+				(font
+					(size 1.27 1.27)
+				)
+				(hide yes)
+			)
+		)
+		(property "Value" "+5VA"
+			(at 425.45 162.5599 90)
+			(effects
+				(font
+					(size 1.27 1.27)
+				)
+				(justify left)
+			)
+		)
+		(property "Footprint" ""
+			(at 421.64 162.56 0)
+			(effects
+				(font
+					(size 1.27 1.27)
+				)
+				(hide yes)
+			)
+		)
+		(property "Datasheet" ""
+			(at 421.64 162.56 0)
+			(effects
+				(font
+					(size 1.27 1.27)
+				)
+				(hide yes)
+			)
+		)
+		(property "Description" "Power symbol creates a global label with name \"+5VA\""
+			(at 421.64 162.56 0)
+			(effects
+				(font
+					(size 1.27 1.27)
+				)
+				(hide yes)
+			)
+		)
+		(pin "1"
+		)
+		(instances
+			(project "Atari65XEC070067RevB"
+				(path "/87d66ada-8337-4a7e-bc00-d889029d79b8"
+					(reference "#PWR0186")
+					(unit 1)
+				)
+			)
+		)
+	)
+	(symbol
 		(lib_id "Device:R_Small")
 		(at 472.44 280.67 90)
@@
 			)
 		)
-		(property "Value" "Case"
+		(property "Value" "GND"
 			(at 38.1 101.6 0)
 			(effects
@@
 			)
 		)
-		(property "Value" "+5VC"
+		(property "Value" "+5VA"
 			(at 21.59 36.83 0)
 			(effects
@@
 	)
 	(symbol
+		(lib_id "Device:R_Small")
+		(at 419.1 162.56 90)
+		(unit 1)
+		(exclude_from_sim no)
+		(in_bom yes)
+		(on_board yes)
+		(dnp no)
+		(property "Reference" "R88"
+			(at 420.878 160.528 90)
+			(effects
+				(font
+					(size 1.27 1.27)
+				)
+				(justify left)
+			)
+		)
+		(property "Value" "3k"
+			(at 420.116 165.354 90)
+			(effects
+				(font
+					(size 1.27 1.27)
+				)
+				(justify left)
+			)
+		)
+		(property "Footprint" "Library:R_Axial_L9.0mm_D2.7mm_P12.70mm_Horizontal"
+			(at 419.1 162.56 0)
+			(effects
+				(font
+					(size 1.27 1.27)
+				)
+				(hide yes)
+			)
+		)
+		(property "Datasheet" "~"
+			(at 419.1 162.56 0)
+			(effects
+				(font
+					(size 1.27 1.27)
+				)
+				(hide yes)
+			)
+		)
+		(property "Description" "Resistor, small symbol"
+			(at 419.1 162.56 0)
+			(effects
+				(font
+					(size 1.27 1.27)
+				)
+				(hide yes)
+			)
+		)
+		(pin "1"
+		)
+		(pin "2"
+		)
+		(instances
+			(project "Atari65XEC070067RevB"
+				(path "/87d66ada-8337-4a7e-bc00-d889029d79b8"
+					(reference "R88")
+					(unit 1)
+				)
+			)
+		)
+	)
+	(symbol
 		(lib_id "power:GND")
 		(at 160.02 27.94 0)
@@
 	(symbol
 		(lib_id "Device:C_Small")
-		(at 288.29 199.39 90)
+		(at 288.29 201.93 90)
 		(unit 1)
 		(exclude_from_sim no)
@@
 		(dnp no)
 		(property "Reference" "C200"
-			(at 288.29 196.85 90)
+			(at 288.29 199.39 90)
 			(effects
 				(font
@@
 		)
 		(property "Value" "100nF"
-			(at 288.29 201.93 90)
+			(at 288.29 204.47 90)
 			(effects
 				(font
@@
 		)
 		(property "Footprint" "Library:C_Axial_L5.1mm_D2.7mm_P12.72mm_Horizontal"
-			(at 288.29 199.39 0)
+			(at 288.29 201.93 0)
 			(effects
 				(font
@@
 		)
 		(property "Datasheet" "~"
-			(at 288.29 199.39 0)
+			(at 288.29 201.93 0)
 			(effects
 				(font
@@
 		)
 		(property "Description" "Unpolarized capacitor, small symbol"
-			(at 288.29 199.39 0)
+			(at 288.29 201.93 0)
 			(effects
 				(font
