File: IO.kicad_sch (KiCad schematic)
At the start: 0 parts

Commit message: tidy up
Parts:
- added C102, C63, C64, C65, C66, C71, C72, C73, C74, C75, C76, C77, C78, C80, C81, C82, C83, C84, C85, C86, C87, C88, C89, C90, C91, C92, C96, C97, C99: 1nF, Library:C_Axial_L5.1mm_D2.7mm_P12.72mm_Horizontal, symbol Device:C_Small
- added C301, C302, C303, C304: 27pF, Library:C_Disc_D3.0mm_W1.6mm_P3.0mm, symbol Device:C_Small
- added C305, C306, C307, C308, C309, C310: 1nF, Library:C_Disc_D3.0mm_W1.6mm_P3.0mm, symbol Device:C_Small
- added C62, C68, C69, C70, C93: 100nF, Library:C_Axial_L5.1mm_D2.7mm_P12.72mm_Horizontal, symbol Device:C_Small
- added C79: 22uF, Capacitor_THT:CP_Axial_L11.0mm_D5.0mm_P18.00mm_Horizontal, symbol Device:C_Polarized_Small
- added C94, C95: 10nF, Library:C_Axial_L5.1mm_D2.7mm_P12.72mm_Horizontal, symbol Device:C_Small
- added C98: 10uF, Capacitor_THT:CP_Axial_L11.0mm_D5.0mm_P18.00mm_Horizontal, symbol Device:C_Polarized_Small
- added CR5: 1N4148, Diode_THT:D_DO-35_SOD27_P12.70mm_Horizontal, symbol Device:D_Small
- added J1: SIO, Library:DSUB-13_Pins_Horizontal_P2.77x2.84mm_EdgePinOffset7.70mm_Housed_MountingHolesOffset9.12mm, symbol Library:SIO
- added J5, J6: JOY1, Library:DSUB-9_Pins_Horizontal_P2.77x2.54mm_Atari, symbol Connector:DE9_Socket
- added J8: KEYBOARD, Library:KEYBOARD, symbol Library:KEYBOARD
- added L10, L102, L11, L12, L23, L30: FB, Inductor_THT:L_Axial_L7.0mm_D3.3mm_P12.70mm_Horizontal_Fastron_MICC, symbol Device:L_Ferrite
- added L15, L16, L17, L18, L19, L20, L21, L22, L25, L26, L27, L28, L29: 10uH, Inductor_THT:L_Axial_L7.0mm_D3.3mm_P12.70mm_Horizontal_Fastron_MICC, symbol Device:L_Ferrite
- added Q7: MPSA55, Library:TO-92L_Inline_Wide, symbol PCM_Transistor_BJT_AKL:MPSA56
- added R117, R118, R119, R128, R129, R130, R131, R90: 100R, Library:R_Axial_L9.0mm_D2.7mm_P12.70mm_Horizontal, symbol Device:R_Small
- added R120, R121, R122, R123, R124, R125, R126, R127, R132, R133, R134, R135, R136, R95: 220R, Library:R_Axial_L9.0mm_D2.7mm_P12.70mm_Horizontal, symbol Device:R_Small
- added R137, R138, R139, R140, R141, R142, R143, R144, R145, R146, R147, R148, R149, R150, R151, R152, R153: 270R, Library:R_Axial_L9.0mm_D2.7mm_P12.70mm_Horizontal, symbol Device:R_Small
- added R206, R23, R24, R25: 3k3, Library:R_Axial_L9.0mm_D2.7mm_P12.70mm_Horizontal, symbol Device:R_Small
- added R74, R75, R86: 3k, Library:R_Axial_L9.0mm_D2.7mm_P12.70mm_Horizontal, symbol Device:R_Small
- added R76, R77, R78, R79: 1k8, Library:R_Axial_L9.0mm_D2.7mm_P12.70mm_Horizontal, symbol Device:R_Small
- added R80: 1k, Library:R_Axial_L9.0mm_D2.7mm_P12.70mm_Horizontal, symbol Device:R_Small
- added R81, R82, R83, R84, R92, R93, R94: 4k7, Library:R_Axial_L9.0mm_D2.7mm_P12.70mm_Horizontal, symbol Device:R_Small
- added R89, R96: 47k, Library:R_Axial_L9.0mm_D2.7mm_P12.70mm_Horizontal, symbol Device:R_Small
- added R91: 2k7, Library:R_Axial_L9.0mm_D2.7mm_P12.70mm_Horizontal, symbol Device:R_Small
- added U22: C012294/POKEY, Package_DIP:DIP-40_W15.24mm, symbol Library:POKEY
- added U23: C014795 PIA/6520, Package_DIP:DIP-40_W15.24mm, symbol Library:6520
- added U24, U25: 4051, Package_DIP:DIP-16_W7.62mm, symbol Library:4051
- added W1: Jumper_2_Closed, Resistor_THT:R_Axial_DIN0309_L9.0mm_D3.2mm_P12.70mm_Horizontal, symbol Jumper:Jumper_2_Bridged
Connections:
- new net: Q7.2 (B), R91.2
- new net: L11.1, Q7.3 (C)
- new net: C62.2, C98.1, C99.2, L12.2, L25.1, U22.17 (VCC)
- new net: L102.2, L25.2
- new net: C85.2, L29.1, R120.2
- new net: R145.1, U25.13 (X0)
- new net: J8.18, R145.2
- new net: C90.2, L21.1, R125.2
- new net: R117.1, R92.1, U23.40 (CA1)
- new net: R119.1, R94.1, U23.19 (CB2)
- new net: C71.2, L17.1, R76.2
- new net: J6.5, L17.2
- new net: R141.1, U25.1 (X4)
- new net: J8.14, R141.2
- new net: R75.1, U22.10 (P4), W1.1 (A)
- new net: R151.1, U24.5 (X5)
- new net: J8.10, R151.2
- new net: R89.2, U22.25 (~{KR1}), U24.3 (X)
- new net: C73.2, L15.1, R78.2
- new net: J8.23 (OPTION), R136.2
- new net: R124.1, U23.6 (PA4)
- new net: C89.2, L22.1, R124.2
- new net: CR5.2 (A), R137.1, R96.1, U22.16 (~{KR2})
- new net: C88.2, L26.1, R123.2
- new net: J6.4, L26.2
- new net: R150.1, U24.1 (X4)
- new net: U22.22 (~{K1}), U24.10 (B)
- new net: U22.23 (~{K0}), U24.11 (A)
- new net: R149.1, U24.12 (X3)
- new net: R146.1, U24.13 (X0)
- new net: R147.1, U24.14 (X1)
- new net: R148.1, U24.15 (X2)
- new net: R152.1, U24.2 (X6)
- new net: R153.1, U24.4 (X7)
- new net: U22.21 (~{K2}), U24.9 (C)
- new net: U22.18 (~{K5}), U25.9 (C)
- new net: U22.19 (~{K4}), U25.10 (B)
- new net: U22.20 (~{K3}), U25.11 (A)
- new net: R74.1, U22.31 (CS1)
- new net: C302.2, C75.2, J1.2, R128.2
- new net: R118.1, U23.18 (CB1)
- new net: R120.1, U23.2 (PA0)
- new net: R86.2, U23.22 (CS0), U23.24 (CS1)
- new net: R121.1, U23.3 (PA1)
- new net: R91.1, U23.39 (CA2)
- new net: R122.1, U23.4 (PA2)
- new net: R123.1, U23.5 (PA3)
- new net: R125.1, U23.7 (PA5)
- new net: R126.1, U23.8 (PA6)
- new net: R127.1, U23.9 (PA7)
- new net: J5.5, L15.2
- new net: J5.1, L22.2
- new net: J5.2, L21.2
- new net: J5.3, L20.2
- new net: J5.4, L19.2
- new net: J5.6, L23.2
- new net: J5.9, L16.2
- new net: R90.2, U25.3 (X)
- new net: C97.2, L30.1, R132.2
- new net: J6.1, L29.2
- new net: J6.2, L28.2
- new net: J6.3, L27.2
- new net: J6.6, L30.2
- new net: J6.9, L18.2
- new net: C301.2, C76.2, J1.1, R129.2
- new net: C92.2, L19.1, R127.2
- new net: R142.1, U25.12 (X3)
- new net: J8.5, R142.2
- new net: R143.1, U25.15 (X2)
- new net: J8.15, R143.2
- new net: R144.1, U25.14 (X1)
- new net: J8.13, R144.2
- new net: C87.2, L27.1, R122.2
- new net: C72.2, L18.1, R77.2
- new net: C303.2, C77.2, J1.3, R130.2
- new net: J8.8, R148.2
- new net: C74.2, L16.1, R79.2
- new net: C91.2, L20.1, R126.2
- new net: C96.2, L23.1, R133.2
- new net: R139.1, U25.2 (X6)
- new net: R138.1, U25.4 (X7)
- new net: R140.1, U25.5 (X5)
- new net: J8.12, R139.2
- new net: C95.2, J8.2, R95.1
- new net: J8.11, R147.2
- new net: J8.22 (SELECT), R135.2
- new net: J8.20, R137.2
- new net: J8.4, R152.2
- new net: C86.2, L28.1, R121.2
- new net: J8.17, R146.2
- new net: C304.2, C78.2, J1.5, R131.2
- new net: J8.16, R149.2
- new net: J8.19, R150.2
- new net: J8.21 (START), R134.2
- new net: J8.6, R140.2
- new net: J8.7, R138.2
- new net: J8.9, R153.2
- new net +5VA: C68.2, C69.1, C70.1, C93.2, C94.1, CR5.1 (K), J8.1, L10.1, L12.1, Q7.1 (E), R206.2, R23.1, R24.1, R25.1, R74.2, R75.2, R80.1, R81.2, R82.2, R83.2, R84.2, R86.1, R89.1, R92.2, R93.2, R94.2, R95.2, R96.2, U23.20 (VCC), U24.16 (VCC), U25.16 (VCC)
- new net +5VD: C102.2, J5.7, J6.7, L102.1
- new net A0: U22.36 (A0), U23.35 (A0)
- new net A1: U22.35 (A1), U23.36 (A1)
- new net A2: U22.34 (A2)
- new net A3: U22.33 (A3)
- new net AUDIO: R80.2, U22.37 (AUDIO)
- new net Bphi2: U22.7 (O2), U23.25 (O2)
- new net CLOCK_IN: R129.1, R82.1, U22.26 (BCLK)
- new net CLOCK_OUT: R128.1, R81.1, U22.27 (ACLK)
- new net COMMAND: C305.2, C84.1, J1.7, R119.2
- new net D0: U22.38 (D0), U23.33 (D0)
- new net D1: U22.39 (D1), U23.32 (D1)
- new net D2: U22.40 (D2), U23.31 (D2)
- new net D3: U22.2 (D3), U23.30 (D3)
- new net D4: U22.3 (D4), U23.29 (D4)
- new net D5: U22.4 (D5), U23.28 (D5)
- new net D6: U22.5 (D6), U23.27 (D6)
- new net D7: U22.6 (D7), U23.26 (D7)
- new net DATA_IN: R130.1, R83.1, U22.24 (SID)
- new net DATA_OUT: R131.1, R84.1, U22.28 (SOD)
- new net GND: C102.1, C301.1, C302.1, C303.1, C304.1, C305.1, C306.1, C307.1, C308.1, C309.1, C310.1, C62.1, C63.1, C64.1, C65.1, C66.1, C68.1, C69.2, C70.2, C71.1, C72.1, C73.1, C74.1, C75.1, C76.1, C77.1, C78.1, C79.2, C80.1, C81.1, C82.2, C83.2, C84.2, C85.1, C86.1, C87.1, C88.1, C89.1, C90.1, C91.1, C92.1, C93.1, C94.2, C95.1, C96.1, C97.1, C98.2, C99.1, J1.4, J1.6, J5.8, J6.8, J8.3, R90.1, U22.1 (GND), U22.11 (P5), U22.8 (P6), U22.9 (P7), U23.1 (VSS), U24.6 (Inh), U24.7 (VEE), U24.8 (VSS), U25.6 (Inh), U25.7 (VEE), U25.8 (VSS), W1.2 (B)
- new net INTERRUPT: C310.2, C83.1, J1.13, R118.2, R93.1
- new net MOTOR_CONTROL: C306.2, C81.2, J1.8, L11.2
- new net P0: C65.2, R77.1, U22.14 (P0)
- new net P1: C64.2, R76.1, U22.15 (P1)
- new net P2: C66.2, R79.1, U22.12 (P2)
- new net P3: C63.2, R78.1, U22.13 (P3)
- new net PB0: U23.10 (PB0)
- new net PB1: U23.11 (PB1)
- new net PB2: R23.2, U23.12 (PB2)
- new net PB3: R25.2, U23.13 (PB3)
- new net PB4: R24.2, U23.14 (PB4)
- new net PB5: R206.1, U23.15 (PB5)
- new net PB7: U23.17 (PB7)
- new net PROCEED: C307.2, C82.1, J1.9, R117.2
- new net READY_+5V: C308.2, C79.1, C80.2, J1.10, L10.2
- new net RESET: J8.24 (RESET)
- new net R/~{W}: U22.32 (R/~{W}), U23.21 (R/~{W})
- new net S0: R134.1
- new net S1: R135.1
- new net S2: R136.1
- new net SIO_AUDIO: C309.2, J1.11
- new net T0: R132.1
- new net T1: R133.1
- new net ~{IRQ}: U22.29 (~{IRQ}), U23.37 (~{IRQB}), U23.38 (~{IRQA})
- new net ~{PIACS}: U23.23 (~{CS2})
- new net ~{POKEYCS}: U22.30 (~{CS0})
- new net ~{RST}: U23.34 (~{RESET})
- no-connect marks 0 -> 2

Commit message: complete tidy up
Other:
- company: (none) -> Original design by Atari
- title: (none) -> 65XE/130XE - C070065/C070067 rev-B
Changed lines of the file:
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@@
 	(paper "A3")
 	(title_block
-		(date "2025-09-28")
+		(title "65XE/130XE - C070065/C070067 rev-B")
+		(date "2025-09-29")
+		(rev "1.1")
+		(company "Original design by Atari")
+		(comment 1 "Transcribed from work by jer/eightbitter")
 	)
 	(rectangle
