File: clocks.kicad_sch (KiCad schematic)
At the start: 70 parts, among them Q4 2N3904, Q5 2N3904, Q6 2N3904, U10 4164, U11 4164, U12 4164, U13 4164, U14 4164, U15 4164, U16 4164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

Commit message: complete tidy up
Other:
- company: (none) -> Original design by Atari
- title: (none) -> 65XE/130XE - C070065/C070067 rev-B
Changed lines of the file:
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@@
 	(paper "A4")
 	(title_block
-		(date "2025-09-27")
+		(title "65XE/130XE - C070065/C070067 rev-B")
+		(date "2025-09-29")
+		(rev "1.1")
+		(company "Original design by Atari")
+		(comment 1 "Transcribed from work by jer/eightbitter")
 	)
 	(rectangle
