File: power.kicad_sch (KiCad schematic)
At the start: 20 parts, among them J7 DIN-7, SW1 SW_SPDT

Commit message: tidy up
Parts:
- added C200, C201: 100nF, Library:C_Axial_L5.1mm_D2.7mm_P12.72mm_Horizontal, symbol Device:C_Small
- added L4: 22uH, Inductor_THT:L_Axial_L7.0mm_D3.3mm_P12.70mm_Horizontal_Fastron_MICC, symbol Device:L_Ferrite
- added R200: 470k, Library:R_Axial_L9.0mm_D2.7mm_P12.70mm_Horizontal, symbol Device:R_Small
- added R39: 56k, Library:R_Axial_L9.0mm_D2.7mm_P12.70mm_Horizontal, symbol Device:R_Small
- added R40: 100R, Library:R_Axial_L9.0mm_D2.7mm_P12.70mm_Horizontal, symbol Device:R_Small
- added U19: NE555P, Package_DIP:DIP-8_W7.62mm, symbol Library:NE555P
Connections:
- net +5VA: now also C201.2, R39.1, U19.4 (R), U19.8 (VCC)
- net GND: now also C201.1, R200.1, U19.1 (GND)
- new net: C200.1, R200.2, U19.2 (TR), U19.6 (THR)
- new net: L4.2, R40.2
- new net: C200.2, R39.2, R40.1
- new net RESET: L4.1
- new net ~{RST}: U19.3 (Q)
- no-connect marks 1 -> 3
Other:
- note added: "Power Delivery"
- note added: "Reset"
- moved on the sheet: C1, C10, C11, C12, C13, C14, C15, C2, C3, C4, C5, C6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

Commit message: complete tidy up
Other:
- company: (none) -> Original design by Atari
- title: (none) -> 65XE/130XE - C070065/C070067 rev-B
Changed lines of the file:
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@@
 	(paper "A5")
 	(title_block
-		(date "2025-09-27")
+		(title "65XE/130XE - C070065/C070067 rev-B")
+		(date "2025-09-29")
+		(rev "1.1")
+		(company "Original design by Atari")
+		(comment 1 "Transcribed from work by jer/eightbitter")
 	)
 	(rectangle
