File: rom.kicad_sch (KiCad schematic)
At the start: 14 parts, among them U2 74LS138, U3 MMU, U4 BASIC, U5 OS ROM

Commit message: complete tidy up
Other:
- company: (none) -> Original design by Atari
- title: (none) -> 65XE/130XE - C070065/C070067 rev-B
Changed lines of the file:
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@@
 	(paper "A5")
 	(title_block
-		(date "2025-09-28")
+		(title "65XE/130XE - C070065/C070067 rev-B")
+		(date "2025-09-29")
+		(rev "1.1")
+		(company "Original design by Atari")
+		(comment 1 "Transcribed from work by jer/eightbitter")
 	)
 	(rectangle
