File: video.kicad_sch (KiCad schematic)
At the start: 40 parts, among them Q6 2N3904, U10 4164, U11 4164, U12 4164, U13 4164, U14 4164, U15 4164, U16 4164, U21 74LS74, U26 4164, U27 4164, U28 4164, U29 4164, U30 4164, U31 4164, U32 4164, U33 4164, U36 MMMU, U6 C061991/FREDDIE, U9 4164, Y2 4.33618MHz

Commit message: tidy up
Parts:
- added C101, C105: 100nF, Library:C_Axial_L5.1mm_D2.7mm_P12.72mm_Horizontal, symbol Device:C_Small
- added C113, C114, C115, C116, C117, C118, C119, C120, C34, C35, C36, C37, C38, C39, C40, C41: 100nF, Library:C_Axial_L3.8mm_D2.6mm_P8.89mm_Horizontal, symbol Device:C_Small
- added C32: 18pF, Library:C_Axial_L5.1mm_D2.7mm_P12.72mm_Horizontal, symbol Device:C_Small
- added C33: 10pF, Library:C_Axial_L5.1mm_D2.7mm_P12.72mm_Horizontal, symbol Device:C_Small
- added Q4, Q5: 2N3904, Library:TO-92L_Inline_Wide, symbol PCM_Transistor_BJT_AKL:2N3904
- added R18, R27: 220R, Library:R_Axial_L9.0mm_D2.7mm_P12.70mm_Horizontal, symbol Device:R_Small
- added R26: 2k2, Library:R_Axial_L9.0mm_D2.7mm_P12.70mm_Horizontal, symbol Device:R_Small
- added R28: 910k, Library:R_Axial_L9.0mm_D2.7mm_P12.70mm_Horizontal, symbol Device:R_Small
- added R29: 1M, Library:R_Axial_L9.0mm_D2.7mm_P12.70mm_Horizontal, symbol Device:R_Small
- added U35: 74LS95, Package_DIP:DIP-14_W7.62mm, symbol Library:74LS95
- added YA1: See Note, Crystal:Crystal_HC49-U_Horizontal, symbol PCM_Crystal_AKL:Crystal_Generic
- added YB1: See Note, Oscillator:Oscillator_DIP-14, symbol Library:CXO-DIP14
- renumbered C49 to C103, R16 to R110, R17 to R111, U36 to U34
Connections:
- net +5VA: now also C101.1, C113.2, C114.2, C115.2, C116.2, C117.2, C118.2, C119.2, C120.2, C34.2, C35.2, C36.2, C37.2, C38.2, C39.2, C40.2, C41.2, U35.14 (VCC)
- net CLKIN: now also Q4.1 (E), R18.1, YB1.8 (OUT)
- net GND: now also C101.2, C105.1, C113.1, C114.1, C115.1, C116.1, C117.1, C118.1, C119.1, C120.1, C32.2, C33.2, C34.1, C35.1, C36.1, C37.1, C38.1, C39.1, C40.1, C41.1, R18.2, R27.2, R29.2, U35.2 (A), U35.3 (B), U35.4 (C), U35.5 (D), U35.6 (Mode), U35.7 (GND), U35.8 (CLK2), YB1.7 (GND)
- net HALT: now also U35.1 (SDI)
- net ~{CAS}high: now also U26.15 (~{CAS}), U27.15 (~{CAS}), U28.15 (~{CAS}), U29.15 (~{CAS}), U30.15 (~{CAS}), U31.15 (~{CAS}), U32.15 (~{CAS}), U33.15 (~{CAS})
- net ~{CAS}low: now also U10.15 (~{CAS}), U11.15 (~{CAS}), U12.15 (~{CAS}), U13.15 (~{CAS}), U14.15 (~{CAS}), U15.15 (~{CAS}), U16.15 (~{CAS}), U9.15 (~{CAS})
- net RA5: now reaches U10.10 (A5), U11.10 (A5), U12.10 (A5), U13.10 (A5), U14.10 (A5), U15.10 (A5), U16.10 (A5), U26.10 (A5), U27.10 (A5), U28.10 (A5), U29.10 (A5), U30.10 (A5), U31.10 (A5), U32.10 (A5), U33.10 (A5), U9.10 (A5)
- net RA5: now also U6.27 (RA5)
- net RA4: now reaches U10.11 (A4), U11.11 (A4), U12.11 (A4), U13.11 (A4), U14.11 (A4), U15.11 (A4), U16.11 (A4), U26.11 (A4), U27.11 (A4), U28.11 (A4), U29.11 (A4), U30.11 (A4), U31.11 (A4), U32.11 (A4), U33.11 (A4), U9.11 (A4)
- net RA4: now also U6.28 (RA4)
- net RA3: now reaches U10.12 (A3), U11.12 (A3), U12.12 (A3), U13.12 (A3), U14.12 (A3), U15.12 (A3), U16.12 (A3), U26.12 (A3), U27.12 (A3), U28.12 (A3), U29.12 (A3), U30.12 (A3), U31.12 (A3), U32.12 (A3), U33.12 (A3), U9.12 (A3)
- net RA3: now also U6.29 (RA3)
- net RA6: now reaches U10.13 (A6), U11.13 (A6), U12.13 (A6), U13.13 (A6), U14.13 (A6), U15.13 (A6), U16.13 (A6), U26.13 (A6), U27.13 (A6), U28.13 (A6), U29.13 (A6), U30.13 (A6), U31.13 (A6), U32.13 (A6), U33.13 (A6), U9.13 (A6)
- net RA6: now also U6.26 (RA6)
- net D2: now reaches U28.14 (DO), U28.2 (DI)
- net D2: now also U11.14 (DO), U11.2 (DI)
- net ~{WE}: now reaches U10.3 (~{WE}), U11.3 (~{WE}), U12.3 (~{WE}), U13.3 (~{WE}), U14.3 (~{WE}), U15.3 (~{WE}), U16.3 (~{WE}), U26.3 (~{WE}), U27.3 (~{WE}), U28.3 (~{WE}), U29.3 (~{WE}), U30.3 (~{WE}), U31.3 (~{WE}), U32.3 (~{WE}), U33.3 (~{WE}), U9.3 (~{WE})
- net ~{WE}: now also U6.34 (~{WRT})
- net ~{RAS}: now reaches U10.4 (~{RAS}), U11.4 (~{RAS}), U12.4 (~{RAS}), U13.4 (~{RAS}), U14.4 (~{RAS}), U15.4 (~{RAS}), U16.4 (~{RAS}), U26.4 (~{RAS}), U27.4 (~{RAS}), U28.4 (~{RAS}), U29.4 (~{RAS}), U30.4 (~{RAS}), U31.4 (~{RAS}), U32.4 (~{RAS}), U33.4 (~{RAS}), U9.4 (~{RAS})
- net ~{RAS}: now also U6.33 (~{RAS})
- net RA0: now reaches U10.5 (A0), U11.5 (A0), U12.5 (A0), U13.5 (A0), U14.5 (A0), U15.5 (A0), U16.5 (A0), U26.5 (A0), U27.5 (A0), U28.5 (A0), U29.5 (A0), U30.5 (A0), U31.5 (A0), U32.5 (A0), U33.5 (A0), U9.5 (A0)
- net RA0: now also U6.32 (RA0)
- net RA2: now reaches U10.6 (A2), U11.6 (A2), U12.6 (A2), U13.6 (A2), U14.6 (A2), U15.6 (A2), U16.6 (A2), U26.6 (A2), U27.6 (A2), U28.6 (A2), U29.6 (A2), U30.6 (A2), U31.6 (A2), U32.6 (A2), U33.6 (A2), U9.6 (A2)
- net RA2: now also U6.30 (RA2)
- net RA1: now reaches U10.7 (A1), U11.7 (A1), U12.7 (A1), U13.7 (A1), U14.7 (A1), U15.7 (A1), U16.7 (A1), U26.7 (A1), U27.7 (A1), U28.7 (A1), U29.7 (A1), U30.7 (A1), U31.7 (A1), U32.7 (A1), U33.7 (A1), U9.7 (A1)
- net RA1: now also U6.31 (RA1)
- net RA7: now reaches U10.9 (A7), U11.9 (A7), U12.9 (A7), U13.9 (A7), U14.9 (A7), U15.9 (A7), U16.9 (A7), U26.9 (A7), U27.9 (A7), U28.9 (A7), U29.9 (A7), U30.9 (A7), U31.9 (A7), U32.9 (A7), U33.9 (A7), U9.9 (A7)
- net RA7: now also U6.25 (RA7)
- net D1: now reaches U10.14 (DO), U10.2 (DI)
- net D1: now also U27.14 (DO), U27.2 (DI)
- net D5: now reaches U14.14 (DO), U14.2 (DI)
- net D5: now also U31.14 (DO), U31.2 (DI)
- net D0: now reaches U26.14 (DO), U26.2 (DI)
- net D0: now also U9.14 (DO), U9.2 (DI)
- net D4: now reaches U13.14 (DO), U13.2 (DI)
- net D4: now also U30.14 (DO), U30.2 (DI)
- net Phi2: now reaches U6.5 (O2)
- net Phi2: now also U34.19 (O2)
- net D6: now reaches U15.14 (DO), U15.2 (DI)
- net D6: now also U32.14 (DO), U32.2 (DI)
- net D7: now reaches U16.14 (DO), U16.2 (DI)
- net D7: now also U33.14 (DO), U33.2 (DI)
- net D3: now reaches U29.14 (DO), U29.2 (DI)
- net D3: now also U12.14 (DO), U12.2 (DI)
- net MHALT: now reaches U34.11 (MHALT)
- net MHALT: now also U35.13 (QA)
- new net: C32.1, Q5.2 (B), R28.2, R29.1, YA1.1
- new net: C33.1, Q4.2 (B), Q5.3 (C), R26.2, YA1.2
- new net: Q5.1 (E), R27.1
- new net +5VB: C105.2, Q4.3 (C), R26.1, R28.1, YB1.14 (Vcc)
- new net Bphi2: U35.9 (CLK1)
- no-connect marks 0 -> 1
Other:
- note added: "!"
- note added: "ALTERNATE TO"
- note added: "U35 IS AN ALTERNATIVE FOR THE CUSTOM GATE ARRAY AND MUST BE USED IN COMBINATION WITH PAL16L8 OR GAL16V8 https://atarimax.com/jindroush.atari.org/data/achips/co25953-pal16l8.vhd"
- note added: "Y1 NTSC - 14.31818 MHz PAL - 14.187576 MHz"
- moved on the sheet: C103, C111, C206, C29, C58, C59, C60, C61, L103, L4, L8, Q6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

Commit message: tidy up
Parts:
- renumbered L4 to L37
Changed lines of the file:
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@@
 		(on_board yes)
 		(dnp no)
-		(property "Reference" "L4"
+		(property "Reference" "L37"
 			(at 85.09 129.032 90)
 			(effects
@@
 			(project "Atari65XEC070067RevB"
 				(path "/87d66ada-8337-4a7e-bc00-d889029d79b8/79b7fc1a-e1af-46b4-bad7-4b1e519c1eac"
-					(reference "L4")
+					(reference "L37")
 					(unit 1)
 				)

Commit message: tidy up video
Parts:
- removed C101, C103, C105, C29, C58, C61: 100nF, Library:C_Axial_L5.1mm_D2.7mm_P12.72mm_Horizontal, symbol Device:C_Small
- removed C111: 820pF, Library:C_Axial_L5.1mm_D2.7mm_P12.72mm_Horizontal, symbol Device:C_Small
- removed C113, C114, C115, C116, C117, C118, C119, C120, C34, C35, C36, C37, C38, C39, C40, C41: 100nF, Library:C_Axial_L3.8mm_D2.6mm_P8.89mm_Horizontal, symbol Device:C_Small
- removed C206: 27pF, Library:C_Axial_L5.1mm_D2.7mm_P12.72mm_Horizontal, symbol Device:C_Small
- removed C32: 18pF, Library:C_Axial_L5.1mm_D2.7mm_P12.72mm_Horizontal, symbol Device:C_Small
- removed C33: 10pF, Library:C_Axial_L5.1mm_D2.7mm_P12.72mm_Horizontal, symbol Device:C_Small
- removed C59: 22pF, Library:C_Axial_L5.1mm_D2.7mm_P12.72mm_Horizontal, symbol Device:C_Small
- removed C60: 56pF, Library:C_Axial_L5.1mm_D2.7mm_P12.72mm_Horizontal, symbol Device:C_Small
- removed L103: 100uH, Inductor_THT:L_Axial_L7.0mm_D3.3mm_P12.70mm_Horizontal_Fastron_MICC, symbol Device:L_Ferrite
- removed L37: FB or 470R, Library:R_Axial_L9.0mm_D2.7mm_P12.70mm_Horizontal, symbol Device:L_Ferrite
- removed L8: 15uH, Library:R_Axial_L9.0mm_D2.7mm_P12.70mm_Horizontal, symbol Device:L_Ferrite
- removed Q4, Q5, Q6: 2N3904, Library:TO-92L_Inline_Wide, symbol PCM_Transistor_BJT_AKL:2N3904
- removed R110, R111: 33R, Library:R_Axial_L9.0mm_D2.7mm_P12.70mm_Horizontal, symbol Device:R_Small
- removed R18, R27: 220R, Library:R_Axial_L9.0mm_D2.7mm_P12.70mm_Horizontal, symbol Device:R_Small
- removed R26: 2k2, Library:R_Axial_L9.0mm_D2.7mm_P12.70mm_Horizontal, symbol Device:R_Small
- removed R28: 910k, Library:R_Axial_L9.0mm_D2.7mm_P12.70mm_Horizontal, symbol Device:R_Small
- removed R29: 1M, Library:R_Axial_L9.0mm_D2.7mm_P12.70mm_Horizontal, symbol Device:R_Small
- removed R69: 6k8, Library:R_Axial_L9.0mm_D2.7mm_P12.70mm_Horizontal, symbol Device:R_Small
- removed R70: 10k, Library:R_Axial_L9.0mm_D2.7mm_P12.70mm_Horizontal, symbol Device:R_Small
- removed R71: 470R, Library:R_Axial_L9.0mm_D2.7mm_P12.70mm_Horizontal, symbol Device:R_Small
- removed R72, R73: 1k, Library:R_Axial_L9.0mm_D2.7mm_P12.70mm_Horizontal, symbol Device:R_Small
- removed U10, U11, U12, U13, U14, U15, U16, U26, U27, U28, U29, U30, U31, U32, U33, U9: 4164, Package_DIP:DIP-16_W7.62mm, symbol Library:4164
- removed U21: 74LS74, Package_DIP:DIP-14_W7.62mm, symbol Library:74LS74
- removed U34: MMMU, Package_DIP:DIP-20_W7.62mm, symbol Library:MMMU
- removed U35: 74LS95, Package_DIP:DIP-14_W7.62mm, symbol Library:74LS95
- removed U6: C061991/FREDDIE, Package_DIP:DIP-40_W15.24mm, symbol Library:FREDDIE
- removed W2: Jumper_2_Open, Resistor_THT:R_Axial_DIN0309_L9.0mm_D3.2mm_P12.70mm_Horizontal, symbol Jumper:Jumper_2_Open
- removed Y2: 4.33618MHz, Crystal:Crystal_HC49-U_Horizontal, symbol PCM_Crystal_AKL:Crystal_Generic
- removed YA1: See Note, Crystal:Crystal_HC49-U_Horizontal, symbol PCM_Crystal_AKL:Crystal_Generic
- removed YB1: See Note, Oscillator:Oscillator_DIP-14, symbol Library:CXO-DIP14
- added A1: ~, Library:RF_Modulator_MDG-UB360S, symbol Library:RF_MOD.
- added C112, C21, C45, C46, C47, C48: 1nF, Library:C_Axial_L5.1mm_D2.7mm_P12.72mm_Horizontal, symbol Device:C_Small
- added C16, C30, C42, C43, C51: 100nF, Library:C_Axial_L5.1mm_D2.7mm_P12.72mm_Horizontal, symbol Device:C_Small
- added C17, C23: 47nF, Library:C_Axial_L5.1mm_D2.7mm_P12.72mm_Horizontal, symbol Device:C_Small
- added C19, C20, C22: 4u7^{*}, Library:CE_NP_Radial_D8.0mm_P2.50mm, symbol Device:C_Small
- added C204, C205: 1uF, Library:C_Axial_L5.1mm_D2.7mm_P12.72mm_Horizontal, symbol Device:C_Small
- added C24: 10uF, Capacitor_THT:CP_Axial_L10.0mm_D4.5mm_P15.00mm_Horizontal, symbol Device:C_Small
- added C25: 150pF, Library:C_Axial_L5.1mm_D2.7mm_P12.72mm_Horizontal, symbol Device:C_Small
- added C44: 68pF, Library:C_Axial_L5.1mm_D2.7mm_P12.72mm_Horizontal, symbol Device:C_Small
- added C50: 10uF, Capacitor_THT:CP_Radial_D5.0mm_P2.50mm, symbol Device:C_Polarized_Small
- added CR2, CR3, CR4: 1N4148, Diode_THT:D_DO-35_SOD27_P12.70mm_Horizontal, symbol Device:D_Small
- added J2: MONITOR, Library:CUI_SDS-50J, symbol Connector:DIN-5_180degree
- added L13: 1.5uH, Inductor_THT:L_Axial_L7.0mm_D3.3mm_P12.70mm_Horizontal_Fastron_MICC, symbol Device:L_Ferrite
- added L31, L5, L7, L9: FB, Inductor_THT:L_Axial_L7.0mm_D3.3mm_P12.70mm_Horizontal_Fastron_MICC, symbol Device:L_Ferrite
- added L32, L6: 100uH, Inductor_THT:L_Axial_L7.0mm_D3.3mm_P12.70mm_Horizontal_Fastron_MICC, symbol Device:L_Ferrite
- added Q1, Q2, Q3: 2N3904, Library:TO-92L_Inline_Wide, symbol PCM_Transistor_BJT_AKL:2N3904
- added R1: 22k, Library:R_Axial_L9.0mm_D2.7mm_P12.70mm_Horizontal, symbol Device:R_Small
- added R10: 10k, Library:R_Axial_L9.0mm_D2.7mm_P12.70mm_Horizontal, symbol Device:R_Small
- added R11: 2k2, Library:R_Axial_L9.0mm_D2.7mm_P12.70mm_Horizontal, symbol Device:R_Small
- added R116: 51R, Library:R_Axial_L9.0mm_D2.7mm_P12.70mm_Horizontal, symbol Device:R_Small
- added R19, R20, R31, R33: 3k, Library:R_Axial_L9.0mm_D2.7mm_P12.70mm_Horizontal, symbol Device:R_Small
- added R2, R52, R7: 2k, Library:R_Axial_L9.0mm_D2.7mm_P12.70mm_Horizontal, symbol Device:R_Small
- added R201: 6k8, Library:R_Axial_L9.0mm_D2.7mm_P12.70mm_Horizontal, symbol Device:R_Small
- added R202: 180R, Library:R_Axial_L9.0mm_D2.7mm_P12.70mm_Horizontal, symbol Device:R_Small
- added R203, R9: 3k3, Library:R_Axial_L9.0mm_D2.7mm_P12.70mm_Horizontal, symbol Device:R_Small
- added R204: 47R, Library:R_Axial_L9.0mm_D2.7mm_P12.70mm_Horizontal, symbol Device:R_Small
- added R205: 150R, Library:R_Axial_L9.0mm_D2.7mm_P12.70mm_Horizontal, symbol Device:R_Small
- added R3: 6k2, Library:R_Axial_L9.0mm_D2.7mm_P12.70mm_Horizontal, symbol Device:R_Small
- added R35: 33k, Library:R_Axial_L9.0mm_D2.7mm_P12.70mm_Horizontal, symbol Device:R_Small
- added R36: 680R, Library:R_Axial_L9.0mm_D2.7mm_P12.70mm_Horizontal, symbol Device:R_Small
- added R37, R41, R42, R43, R44, R45: 1k, Library:R_Axial_L9.0mm_D2.7mm_P12.70mm_Horizontal, symbol Device:R_Small
- added R38: 500k, Library:Potentiometer_Bourns_3352E_Vertical, symbol Device:R_Potentiometer_Small
- added R4: 56k, Library:R_Axial_L9.0mm_D2.7mm_P12.70mm_Horizontal, symbol Device:R_Small
- added R46: 1k6, Library:R_Axial_L9.0mm_D2.7mm_P12.70mm_Horizontal, symbol Device:R_Small
- added R47: 36k, Library:R_Axial_L9.0mm_D2.7mm_P12.70mm_Horizontal, symbol Device:R_Small
- added R48: 18k, Library:R_Axial_L9.0mm_D2.7mm_P12.70mm_Horizontal, symbol Device:R_Small
- added R49: 9K1, Library:R_Axial_L9.0mm_D2.7mm_P12.70mm_Horizontal, symbol Device:R_Small
- added R5: 470k, Library:R_Axial_L9.0mm_D2.7mm_P12.70mm_Horizontal, symbol Device:R_Small
- added R50: 4k7, Library:R_Axial_L9.0mm_D2.7mm_P12.70mm_Horizontal, symbol Device:R_Small
- added R51: 750R, Library:R_Axial_L9.0mm_D2.7mm_P12.70mm_Horizontal, symbol Device:R_Small
- added R53: 100R, Library:R_Axial_L9.0mm_D2.7mm_P12.70mm_Horizontal, symbol Device:R_Small
- added R6: 68k, Library:R_Axial_L9.0mm_D2.7mm_P12.70mm_Horizontal, symbol Device:R_Small
- added R8: 5k1, Library:R_Axial_L9.0mm_D2.7mm_P12.70mm_Horizontal, symbol Device:R_Small
- added U1: LM358, Package_DIP:DIP-8_W7.62mm, symbol Amplifier_Operational:LM358
- added U17: C014889/GTIA, Package_DIP:DIP-40_W15.24mm, symbol Library:GTIA
- added U18: 74LS08, Package_DIP:DIP-14_W7.62mm, symbol 74xx:74LS08
- added U20: 4050, Package_DIP:DIP-16_W7.62mm, symbol 4xxx:4050
- added U7: C021698/ANTIC, Package_DIP:DIP-40_W15.24mm, symbol Library:ANTIC
Connections:
- net +5VA: now also C30.1, C42.1, C43.1, CR2.2 (A), L5.2, R19.1, R20.2, R31.1, R33.2, R35.1, R36.1, R41.1, R42.1, R43.1, R44.1, R45.1, U17.27 (VCC), U18.14 (VCC), U20.16 (NC), U7.21 (VCC)
- net A0: now also U17.2 (A0), U7.13 (A0)
- net A1: now also U17.1 (A1), U7.12 (A1)
- net A10: now also U7.16 (A10)
- net A11: now also U7.22 (A11)
- net A12: now also U7.17 (A12)
- net A13: now also U7.18 (A13)
- net A14: now also U7.19 (A14)
- net A15: now also U7.20 (A15)
- net A2: now also U17.40 (A2), U7.11 (A2)
- net A3: now also U17.39 (A3), U7.10 (A3)
- net A4: now also U17.38 (A4), U7.28 (A4)
- net A5: now also U7.27 (A5)
- net A6: now also U7.26 (A6)
- net A7: now also U7.25 (A7)
- net A8: now also U7.24 (A8)
- net A9: now also U7.23 (A9)
- net Bphi2: now also U17.30 (O2)
- net COLOR_OSC: now also U17.28 (OSC)
- net D0: now also U17.7 (D0), U7.30 (D0)
- net D1: now also U17.6 (D1), U7.31 (D1)
- net D2: now also U17.5 (D2), U7.32 (D2)
- net D3: now also U17.4 (D3), U7.33 (D3)
- net D4: now also U17.37 (D4), U7.40 (D4)
- net D5: now also U17.36 (D5), U7.39 (D5)
- net D6: now also U17.35 (D6), U7.38 (D6)
- net D7: now also U17.34 (D7), U7.37 (D7)
- net GND: now also A1.6 (Case), C112.2, C16.2, C204.2, C205.2, C21.2, C24.2, C25.2, C30.2, C42.2, C43.2, C46.1, C47.1, C48.1, C50.2, C51.1, J2.2, Q1.1 (E), R10.1, R11.2, R202.1, R3.1, R38.1, R52.1, R53.1, U1.4 (V-), U17.3 (GND), U18.7 (GND), U20.8 (VSS), U20.9, U7.1 (GND)
- net HALT: now also U17.26 (HALT), U7.9 (~{HALT})
- net PAL: now also U17.16 (PAL)
- net Phi2: now also R20.1, U18.1
- new net: CR4.1 (K), U20.15
- new net: CR4.2 (A), R51.1
- new net: U18.4, U18.5, U7.34 (O0)
- new net: C19.2, C20.1, C21.1, C22.1, R2.2
- new net: Q3.2 (B), R46.1, R47.2, R48.2, R49.2, R50.2, R51.2, R52.2
- new net: C50.1, C51.2, L5.1, R116.2, R46.2, U20.1 (VCC)
- new net: R1.1, R2.1, R3.2, U1.7
- new net: C20.2, R7.1
- new net: A1.5, L7.1
- new net: C45.1, CR2.1 (K), CR3.2 (A)
- new net: C45.2, Q1.3 (C), R36.2
- new net: C46.2, CR3.1 (K), R37.1
- new net: C23.1, R5.2
- new net: U17.32 (~{CS}), U18.8
- new net: L6.2, R201.1
- new net: A1.1, R6.2, R8.2, U1.1
- new net: R5.1, R6.1, R7.2, U1.2 (-)
- new net: C24.1, R11.1, R9.2, U1.3 (+), U1.5 (+)
- new net: L31.1, R205.2
- new net: C48.2, R38.2, U17.17 (CADJ)
- new net: C47.2, R37.2, R38.3
- new net: R50.1, U20.2
- new net: U17.33 (R/~{W}), U7.14 (R/~{W})
- new net: U17.18 (AN0), U7.2 (AN0)
- new net: U18.3, U7.29 (O2)
- new net: U17.19 (AN1), U7.3 (AN1)
- new net: U17.29 (FO0), U7.35 (FO0)
- new net: R33.1, U18.11, U7.4 (LP)
- new net: U17.20 (AN2), U7.5 (AN2)
- new net: R31.2, U7.6 (~{RNMI})
- new net: R49.1, U20.4
- new net: R1.2, R4.2, U1.6 (-)
- new net: Q2.1 (E), R202.2, R205.1
- new net: A1.2, Q3.1 (E), R204.1, R53.2
- new net: Q3.3 (C), R116.1
- new net: R19.2, U18.2
- new net: L9.1, R204.2
- new net: C17.1, R4.1
- new net: A1.4 (Vcc), C205.1, L13.2
- new net: R47.1, U20.6
- new net: C44.2, Q1.2 (B), R35.2
- new net: R48.1, U20.12
- new net: Q2.2 (B), R201.2
- new net: A1.3, L32.1
- new net: L32.2, R203.1
- new net +5VC: C16.1, C204.1, L13.1, Q2.3 (C), R9.1, U1.8 (V+)
- new net AUDIO: C17.2
- new net CHROMA: J2.5, L31.2
- new net COLOR: L6.1, R203.2, R45.2, U17.21 (COLOR)
- new net COMPOSITE: J2.4, L7.2
- new net CSYNC: U17.25 (CSYNC), U20.14
- new net GTIAsel: C25.1, U18.10, U18.9
- new net LUMA: J2.1, L9.2
- new net MONITOR_AUDIO: J2.3, R10.2, R8.1
- new net Phi0Buf: U18.6
- new net Phi1: C44.1
- new net RD5: U17.11 (T3)
- new net RDY: U7.15 (RDY)
- new net S0: U17.12 (S0)
- new net S1: U17.13 (S1)
- new net S2: U17.14 (S2)
- new net S3: C23.2, U17.15 (S3)
- new net SIO_AUDIO: C112.1, C19.1
- new net T0: U17.8 (T0), U18.12
- new net T1: U17.9 (T1), U18.13
- new net Y0: R41.2, U17.31 (LUM0), U20.7
- new net Y1: R42.2, U17.22 (LUM1), U20.11
- new net Y2: R43.2, U17.23 (LUM2), U20.5
- new net Y3: R44.2, U17.24 (LUM3), U20.3
- new net ~{NMI}: U7.7 (~{NMI})
- new net ~{REF}: U7.8 (~{REF})
- no-connect marks 1 -> 2
Other:
- note added: "MODULATOR REQUIREMENTS NSTC - UM1452 PAL B (GERMANY) CH 3/4 PAL I (UK) VE0405"
- note added: "^{*}C19, C20, C22 are non-polarized"
- note removed: "!"
- note removed: "*"
- note removed: "ADD JUMPER FOR W2^{*} FOR NTSC"
- note removed: "ALTERNATE TO"
- note removed: "NOT REQUIRED FOR NTSC"
- note removed: "U35 IS AN ALTERNATIVE FOR THE CUSTOM GATE ARRAY AND MUST BE USED IN COMBINATION WITH PAL16L8 OR GAL16V8 https://atarimax.com/jindroush.atari.org/data/achips/co25953-pal16l8.vhd"
- note removed: "When L37 is a resistor then C206 is not populated"
- note removed: "Y1 NTSC - 14.31818 MHz PAL - 14.187576 MHz"

Commit message: complete tidy up
Connections:
- net Bphi2: now also U18.3, U7.29 (O2)
- net EXT_AUD: now reaches C22.2
- net R/~{W}: now reaches U17.33 (R/~{W}), U7.14 (R/~{W})
- net ~{RST}: now reaches U7.36 (~{RST})
Other:
- company: (none) -> Original design by Atari
- title: (none) -> 65XE/130XE - C070065/C070067 rev-B
- moved on the sheet: U18A
Changed lines of the file:
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@@
 	(paper "A3")
 	(title_block
+		(title "65XE/130XE - C070065/C070067 rev-B")
 		(date "2025-09-29")
+		(rev "1.1")
+		(company "Original design by Atari")
+		(comment 1 "Transcribed from work by jer/eightbitter")
 	)
 	(text "MODULATOR REQUIREMENTS\nNSTC - UM1452\nPAL B (GERMANY) CH 3/4\nPAL I (UK) VE0405"
@@
 	)
 	(junction
+		(at 140.97 184.15)
+		(diameter 0)
+		(color 0 0 0 0)
+	)
+	(junction
 		(at 234.95 115.57)
 		(diameter 0)
@@
 	(wire
 		(pts
-			(xy 172.72 148.59) (xy 168.91 148.59)
+			(xy 123.19 196.85) (xy 124.46 196.85)
 		)
 		(stroke
@@
 	(wire
 		(pts
-			(xy 123.19 196.85) (xy 124.46 196.85)
+			(xy 146.05 143.51) (xy 148.59 143.51)
 		)
 		(stroke
@@
 	(wire
 		(pts
-			(xy 146.05 143.51) (xy 148.59 143.51)
+			(xy 34.29 147.32) (xy 34.29 146.05)
 		)
 		(stroke
@@
 	(wire
 		(pts
-			(xy 34.29 147.32) (xy 34.29 146.05)
+			(xy 168.91 184.15) (xy 187.96 184.15)
 		)
 		(stroke
@@
 	(wire
 		(pts
-			(xy 168.91 184.15) (xy 187.96 184.15)
+			(xy 113.03 114.3) (xy 135.89 114.3)
 		)
 		(stroke
@@
 	(wire
 		(pts
-			(xy 113.03 114.3) (xy 135.89 114.3)
+			(xy 257.81 229.87) (xy 257.81 227.33)
 		)
 		(stroke
@@
 	(wire
 		(pts
-			(xy 257.81 229.87) (xy 257.81 227.33)
+			(xy 161.29 128.27) (xy 168.91 128.27)
 		)
 		(stroke
@@
 	(wire
 		(pts
-			(xy 161.29 128.27) (xy 168.91 128.27)
+			(xy 140.97 184.15) (xy 148.59 184.15)
 		)
 		(stroke
@@
 	(wire
 		(pts
+			(xy 140.97 182.88) (xy 140.97 184.15)
+		)
+		(stroke
+			(width 0)
+			(type default)
+		)
+	)
+	(wire
+		(pts
 			(xy 96.52 193.04) (xy 96.52 194.31)
 		)
@@
 	(wire
 		(pts
-			(xy 123.19 181.61) (xy 127 181.61)
+			(xy 123.19 181.61) (xy 124.46 181.61)
 		)
 		(stroke
@@
 	(wire
 		(pts
-			(xy 127 186.69) (xy 123.19 186.69)
+			(xy 124.46 186.69) (xy 123.19 186.69)
 		)
 		(stroke
@@
 	(wire
 		(pts
-			(xy 142.24 184.15) (xy 148.59 184.15)
+			(xy 139.7 184.15) (xy 140.97 184.15)
 		)
 		(stroke
@@
 		)
 	)
+	(global_label "~{RST}"
+		(shape input)
+		(at 168.91 148.59 0)
+		(fields_autoplaced yes)
+		(effects
+			(font
+				(size 1.27 1.27)
+			)
+			(justify left)
+		)
+		(property "Intersheetrefs" "${INTERSHEET_REFS}"
+			(at 175.3423 148.59 0)
+			(effects
+				(font
+					(size 1.27 1.27)
+				)
+				(justify left)
+				(hide yes)
+			)
+		)
+	)
 	(global_label "~{REF}"
 		(shape input)
@@
 		)
 	)
+	(global_label "R{slash}~{W}"
+		(shape input)
+		(at 177.8 146.05 0)
+		(fields_autoplaced yes)
+		(effects
+			(font
+				(size 1.27 1.27)
+			)
+			(justify left)
+		)
+		(property "Intersheetrefs" "${INTERSHEET_REFS}"
+			(at 184.8371 146.05 0)
+			(effects
+				(font
+					(size 1.27 1.27)
+				)
+				(justify left)
+				(hide yes)
+			)
+		)
+	)
 	(global_label "D[0..7]"
 		(shape bidirectional)
@@
 		)
 	)
+	(global_label "Bphi2"
+		(shape output)
+		(at 140.97 182.88 90)
+		(fields_autoplaced yes)
+		(effects
+			(font
+				(size 1.27 1.27)
+			)
+			(justify left)
+		)
+		(property "Intersheetrefs" "${INTERSHEET_REFS}"
+			(at 140.97 174.5125 90)
+			(effects
+				(font
+					(size 1.27 1.27)
+				)
+				(justify left)
+				(hide yes)
+			)
+		)
+	)
+	(global_label "EXT_AUD"
+		(shape input)
+		(at 57.15 200.66 270)
+		(fields_autoplaced yes)
+		(effects
+			(font
+				(size 1.27 1.27)
+			)
+			(justify right)
+		)
+		(property "Intersheetrefs" "${INTERSHEET_REFS}"
+			(at 57.15 211.628 90)
+			(effects
+				(font
+					(size 1.27 1.27)
+				)
+				(justify right)
+				(hide yes)
+			)
+		)
+	)
 	(global_label "SIO_AUDIO"
 		(shape input)
@@
 	(symbol
 		(lib_id "74xx:74LS08")
-		(at 134.62 184.15 0)
+		(at 132.08 184.15 0)
 		(unit 1)
 		(exclude_from_sim no)
@@
 		(fields_autoplaced yes)
 		(property "Reference" "U18"
-			(at 134.6117 175.26 0)
+			(at 132.0717 175.26 0)
 			(effects
 				(font
@@
 		)
 		(property "Value" "74LS08"
-			(at 134.6117 177.8 0)
+			(at 132.0717 177.8 0)
 			(effects
 				(font
@@
 		)
 		(property "Footprint" "Package_DIP:DIP-14_W7.62mm"
-			(at 134.62 184.15 0)
+			(at 132.08 184.15 0)
 			(effects
 				(font
@@
 		)
 		(property "Datasheet" "http://www.ti.com/lit/gpn/sn74LS08"
-			(at 134.62 184.15 0)
+			(at 132.08 184.15 0)
 			(effects
 				(font
@@
 		)
 		(property "Description" "Quad And2"
-			(at 134.62 184.15 0)
+			(at 132.08 184.15 0)
 			(effects
 				(font
@@
 		)
 		(property "DigiKey" "296-1633-5-ND"
-			(at 134.62 184.15 0)
+			(at 132.08 184.15 0)
 			(effects
 				(font
@@
 		)
 		(property "LCSC" ""
-			(at 134.62 184.15 0)
+			(at 132.08 184.15 0)
 			(effects
 				(font
